Commit message: I added working contact sensor for one leg and update files used during walking tests

File: sim_and_real/ros2_ws_hex/src/hexapod_description/urdf/hexapod_ee.urdf.xacro (robot description, xacro)
@@ -22,4 +22,13 @@
       </plugin>
     </gazebo>
+    <gazebo>
+      <plugin filename="gz-sim-touchplugin-system"
+        name="gz::sim::systems::TouchPlugin">
+          <target>ground_plane</target>
+          <namespace>tip</namespace>
+          <time>0.001</time>
+          <enabled>true</enabled>
+      </plugin>
+    </gazebo>
     <gazebo reference="${prefix}base_link">
       <sensor name="imu_sensor" type="imu">

File: sim_and_real/ros2_ws_hex/src/hexapod_description/urdf/hexapod_leg_ee.urdf.xacro (robot description, xacro)
@@ -362,8 +362,9 @@
   <!-- Macro: Effector Joint -->
   <xacro:macro name="end_effector_joint" params="prefix index xyz rpy">
-    <joint name="${prefix}joint4_${index}" type="fixed">
+    <joint name="${prefix}joint4_${index}" type="revolute">
       <parent link="${prefix}link4_${index}"/>
       <child link="${prefix}link5_${index}"/>
       <origin xyz="${xyz}" rpy="${rpy}"/>
+      <limit effort="5.0" velocity="1.0" lower="0" upper="0"/>
     </joint>
   </xacro:macro>

Commit message: correction to previous commit

File: sim_and_real/ros2_ws_hex/src/hexapod_description/urdf/hexapod_ee.urdf.xacro (robot description, xacro)
@@ -31,4 +31,11 @@
       </plugin>
     </gazebo>
+    <gazebo reference="${prefix}link5_1">
+      <sensor name='sensor_contact_1' type='contact'>
+          <contact>
+              <collision>link5_1_collision</collision>
+          </contact>
+      </sensor>
+    </gazebo>
     <gazebo reference="${prefix}base_link">
       <sensor name="imu_sensor" type="imu">
