Commit message: Contact sensors for all legs are working. Now they publish ros2 topic that gives information about contact

File: sim_and_real/ros2_ws_hex/src/hexapod_description/urdf/hexapod_leg_ee.urdf.xacro (robot description, xacro)
@@ -132,4 +132,12 @@
       <xacro:property name="joint3_lower" value="-0.523598776"/>
       <xacro:property name="joint3_upper" value="1.570796327"/>
+      <!-- MOMENTY OBROTOWE SERW -->
+      <xacro:property name="joint1_effort" value="2.548"/>
+      <xacro:property name="joint2_effort" value="1.911"/>
+      <xacro:property name="joint3_effort" value="1.911"/>
+      <!-- PRĘDKOŚCI MAKSYMALNE SERW -->
+      <xacro:property name="joint1_velocity" value="3.1"/>
+      <xacro:property name="joint2_velocity" value="4.1"/>
+      <xacro:property name="joint3_velocity" value="4.1"/>
       <!-- CECHY POŁOŻENIA STAWÓW LEG 1 -->
       <xacro:property name="joint1_1_xyz" value="0.086185	0.0860902	0.0170504"/>
@@ -289,5 +297,5 @@
       </xacro:macro>
     <!-- Macro: Joint -->
-    <xacro:macro name="leg_joint" params="prefix joint_name parent_link child_link xyz axis lower upper">
+    <xacro:macro name="leg_joint" params="prefix joint_name parent_link child_link xyz axis lower upper effort velocity">
       <joint name="${joint_name}" type="revolute">
         <parent link="${parent_link}"/>
@@ -295,5 +303,5 @@
         <origin xyz="${xyz}" rpy="0 0 0"/>
         <axis xyz="${axis}"/>
-        <limit effort="5.0" velocity="1.0" lower="${lower}" upper="${upper}"/>
+        <limit effort="${effort}" velocity="${velocity}" lower="${lower}" upper="${upper}"/>
         <dynamics damping="0.1"/>
       </joint>
@@ -411,5 +419,7 @@
       axis="${joint1_1_axis}"
       lower="${joint1_lower}"
-      upper="${joint1_upper}" />
+      upper="${joint1_upper}"
+      effort="${joint1_effort}"
+      velocity="${joint1_velocity}"/>
     <xacro:upper_leg prefix="${prefix}" index="1" xyz="${link2_1_xyz}" rpy="${link2_1_rpy}" />
     <xacro:leg_joint
@@ -421,5 +431,7 @@
       axis="${joint2_1_axis}"
       lower="${joint2_lower}"
-      upper="${joint2_upper}" />
+      upper="${joint2_upper}"
+      effort="${joint2_effort}"
+      velocity="${joint2_velocity}"/>
     <xacro:mid_leg prefix="${prefix}" index="1" xyz="${link3_1_xyz}" rpy="${link3_1_rpy}" />
     <xacro:leg_joint
@@ -431,5 +443,7 @@
       axis="${joint3_1_axis}"
       lower="${joint3_lower}"
-      upper="${joint3_upper}" />
+      upper="${joint3_upper}"
+      effort="${joint3_effort}"
+      velocity="${joint3_velocity}"/>
     <xacro:lower_leg prefix="${prefix}" index="1" xyz="${link4_1_xyz}" rpy="${link4_1_rpy}" />
     <xacro:end_effector_joint prefix="${prefix}" index="1" xyz="${joint4_1_xyz}" rpy="${joint4_1_axis}"/>
@@ -449,5 +463,7 @@
       axis="${joint1_2_axis}"
       lower="${joint1_lower}"
-      upper="${joint1_upper}"/>
+      upper="${joint1_upper}"
+      effort="${joint1_effort}"
+      velocity="${joint1_velocity}"/>
     <xacro:upper_leg prefix="${prefix}" index="2" xyz="${link2_2_xyz}" rpy="${link2_2_rpy}"/>
     <xacro:leg_joint
@@ -459,5 +475,7 @@
       axis="${joint2_2_axis}"
       lower="${joint2_lower}"
-      upper="${joint2_upper}"/>
+      upper="${joint2_upper}"
+      effort="${joint2_effort}"
+      velocity="${joint2_velocity}"/>
     <xacro:mid_leg prefix="${prefix}" index="2" xyz="${link3_2_xyz}" rpy="${link3_2_rpy}"/>
     <xacro:leg_joint
@@ -469,5 +487,7 @@
       axis="${joint3_2_axis}"
       lower="${joint3_lower}"
-      upper="${joint3_upper}"/>
+      upper="${joint3_upper}"
+      effort="${joint3_effort}"
+      velocity="${joint3_velocity}"/>
     <xacro:lower_leg prefix="${prefix}" index="2" xyz="${link4_2_xyz}" rpy="${link4_2_rpy}"/>
     <xacro:end_effector_joint prefix="${prefix}" index="2" xyz="${joint4_2_xyz}" rpy="${joint4_2_axis}"/>
@@ -487,5 +507,7 @@
       axis="${joint1_3_axis}"
       lower="${joint1_lower}"
-      upper="${joint1_upper}"/>
+      upper="${joint1_upper}"
+      effort="${joint1_effort}"
+      velocity="${joint1_velocity}"/>
     <xacro:upper_leg prefix="${prefix}" index="3" xyz="${link2_3_xyz}" rpy="${link2_3_rpy}"/>
     <xacro:leg_joint
@@ -497,5 +519,7 @@
       axis="${joint2_3_axis}"
       lower="${joint2_lower}"
-      upper="${joint2_upper}"/>
+      upper="${joint2_upper}"
+      effort="${joint2_effort}"
+      velocity="${joint2_velocity}"/>
     <xacro:mid_leg prefix="${prefix}" index="3" xyz="${link3_3_xyz}" rpy="${link3_3_rpy}"/>
     <xacro:leg_joint
@@ -507,5 +531,7 @@
       axis="${joint3_3_axis}"
       lower="${joint3_lower}"
-      upper="${joint3_upper}"/>
+      upper="${joint3_upper}"
+      effort="${joint3_effort}"
+      velocity="${joint3_velocity}"/>
     <xacro:lower_leg prefix="${prefix}" index="3" xyz="${link4_3_xyz}" rpy="${link4_3_rpy}"/>
     <xacro:end_effector_joint prefix="${prefix}" index="3" xyz="${joint4_3_xyz}" rpy="${joint4_3_axis}"/>
@@ -525,5 +551,7 @@
       axis="${joint1_4_axis}"
       lower="${joint1_lower}"
-      upper="${joint1_upper}"/>
+      upper="${joint1_upper}"
+      effort="${joint1_effort}"
+      velocity="${joint1_velocity}"/>
     <xacro:upper_leg prefix="${prefix}" index="4" xyz="${link2_4_xyz}" rpy="${link2_4_rpy}"/>
     <xacro:leg_joint
@@ -535,5 +563,7 @@
       axis="${joint2_4_axis}"
       lower="${joint2_lower}"
-      upper="${joint2_upper}"/>
+      upper="${joint2_upper}"
+      effort="${joint2_effort}"
+      velocity="${joint2_velocity}"/>
     <xacro:mid_leg prefix="${prefix}" index="4" xyz="${link3_4_xyz}" rpy="${link3_4_rpy}"/>
     <xacro:leg_joint
@@ -545,5 +575,7 @@
       axis="${joint3_4_axis}"
       lower="${joint3_lower}"
-      upper="${joint3_upper}"/>
+      upper="${joint3_upper}"
+      effort="${joint3_effort}"
+      velocity="${joint3_velocity}"/>
     <xacro:lower_leg prefix="${prefix}" index="4" xyz="${link4_4_xyz}" rpy="${link4_4_rpy}"/>
     <xacro:end_effector_joint prefix="${prefix}" index="4" xyz="${joint4_4_xyz}" rpy="${joint4_4_axis}"/>
@@ -563,5 +595,7 @@
       axis="${joint1_5_axis}"
       lower="${joint1_lower}"
-      upper="${joint1_upper}"/>
+      upper="${joint1_upper}"
+      effort="${joint1_effort}"
+      velocity="${joint1_velocity}"/>
     <xacro:upper_leg prefix="${prefix}" index="5" xyz="${link2_5_xyz}" rpy="${link2_5_rpy}"/>
     <xacro:leg_joint
@@ -573,5 +607,7 @@
       axis="${joint2_5_axis}"
       lower="${joint2_lower}"
-      upper="${joint2_upper}"/>
+      upper="${joint2_upper}"
+      effort="${joint2_effort}"
+      velocity="${joint2_velocity}"/>
     <xacro:mid_leg prefix="${prefix}" index="5" xyz="${link3_5_xyz}" rpy="${link3_5_rpy}"/>
     <xacro:leg_joint
@@ -583,5 +619,7 @@
       axis="${joint3_5_axis}"
       lower="${joint3_lower}"
-      upper="${joint3_upper}"/>
+      upper="${joint3_upper}"
+      effort="${joint3_effort}"
+      velocity="${joint3_velocity}"/>
     <xacro:lower_leg prefix="${prefix}" index="5" xyz="${link4_5_xyz}" rpy="${link4_5_rpy}"/>
     <xacro:end_effector_joint prefix="${prefix}" index="5" xyz="${joint4_5_xyz}" rpy="${joint4_5_axis}"/>
@@ -601,5 +639,7 @@
       axis="${joint1_6_axis}"
       lower="${joint1_lower}"
-      upper="${joint1_upper}"/>
+      upper="${joint1_upper}"
+      effort="${joint1_effort}"
+      velocity="${joint1_velocity}"/>
     <xacro:upper_leg prefix="${prefix}" index="6" xyz="${link2_6_xyz}" rpy="${link2_6_rpy}"/>
     <xacro:leg_joint
@@ -611,5 +651,7 @@
       axis="${joint2_6_axis}"
       lower="${joint2_lower}"
-      upper="${joint2_upper}"/>
+      upper="${joint2_upper}"
+      effort="${joint2_effort}"
+      velocity="${joint2_velocity}"/>
     <xacro:mid_leg prefix="${prefix}" index="6" xyz="${link3_6_xyz}" rpy="${link3_6_rpy}"/>
     <xacro:leg_joint
@@ -621,5 +663,7 @@
       axis="${joint3_6_axis}"
       lower="${joint3_lower}"
-      upper="${joint3_upper}"/>
+      upper="${joint3_upper}"
+      effort="${joint3_effort}"
+      velocity="${joint3_velocity}"/>
     <xacro:lower_leg prefix="${prefix}" index="6" xyz="${link4_6_xyz}" rpy="${link4_6_rpy}"/>
     <xacro:end_effector_joint prefix="${prefix}" index="6" xyz="${joint4_6_xyz}" rpy="${joint4_6_axis}"/>

File: sim_and_real/ros2_ws_hex/src/hexapod_moveit_config/config/hexapod.ros2_control.xacro (robot description, xacro)
@@ -52,4 +52,8 @@
                 <state_interface name="velocity"/>
             </joint>
+            <joint name="joint4_1">
+                <command_interface name="position"/>
+                <state_interface name="position"/>
+            </joint>
             <!-- Leg 2 joints -->
             <joint name="joint1_2">
@@ -73,4 +77,8 @@
                 </state_interface>
                 <state_interface name="velocity"/>
+            </joint>
+            <joint name="joint4_2">
+                <command_interface name="position"/>
+                <state_interface name="position"/>
             </joint>
             <!-- Leg 3 joints -->
@@ -96,4 +104,8 @@
                 <state_interface name="velocity"/>
             </joint>
+            <joint name="joint4_3">
+                <command_interface name="position"/>
+                <state_interface name="position"/>
+            </joint>
             <!-- Leg 4 joints -->
             <joint name="joint1_4">
@@ -117,4 +129,8 @@
                 </state_interface>
                 <state_interface name="velocity"/>
+            </joint>
+            <joint name="joint4_4">
+                <command_interface name="position"/>
+                <state_interface name="position"/>
             </joint>
             <!-- Leg 5 joints -->
@@ -140,4 +156,8 @@
                 <state_interface name="velocity"/>
             </joint>
+            <joint name="joint4_5">
+                <command_interface name="position"/>
+                <state_interface name="position"/>
+            </joint>
             <!-- Leg 6 joints -->
             <joint name="joint1_6">
@@ -162,4 +182,8 @@
                 <state_interface name="velocity"/>
             </joint>
+            <joint name="joint4_6">
+                <command_interface name="position"/>
+                <state_interface name="position"/>
+            </joint>
         </ros2_control>
     </xacro:macro>
