Commit message: IMU in gazebo is working

File: sim_and_real/ros2_ws_hex/src/hexapod_description/gazebo/hexapod.gazebo.xacro (robot description, xacro)
@@ -24,4 +24,15 @@
     </gazebo>
   </xacro:macro>
+  <!-- Gazebo reference for end effector link -->
+   <xacro:macro name="EndEffectorLink" params="reference">
+    <gazebo reference="${reference}">
+      <kp>1000000.0</kp>
+      <kd>100.0</kd>
+      <mu1>30.0</mu1>
+      <mu2>30.0</mu2>
+      <maxVel>1.0</maxVel>
+      <minDepth>0.001</minDepth>
+    </gazebo>
+   </xacro:macro>
   <!-- Define links for all parts of the hexapod -->
   <xacro:Link reference="${prefix}base_link"/>
@@ -31,4 +42,5 @@
   <xacro:Link reference="${prefix}link3_1"/>
   <xacro:Link reference="${prefix}link4_1"/>
+  <xacro:EndEffectorLink reference="${prefix}link5_1"/>
   <!-- Leg 2 links -->
   <xacro:Link reference="${prefix}link1_2"/>
@@ -36,4 +48,5 @@
   <xacro:Link reference="${prefix}link3_2"/>
   <xacro:Link reference="${prefix}link4_2"/>
+  <xacro:EndEffectorLink reference="${prefix}link5_2"/>
   <!-- Leg 3 links -->
   <xacro:Link reference="${prefix}link1_3"/>
@@ -41,4 +54,5 @@
   <xacro:Link reference="${prefix}link3_3"/>
   <xacro:Link reference="${prefix}link4_3"/>
+  <xacro:EndEffectorLink reference="${prefix}link5_3"/>
   <!-- Leg 4 links -->
   <xacro:Link reference="${prefix}link1_4"/>
@@ -46,4 +60,5 @@
   <xacro:Link reference="${prefix}link3_4"/>
   <xacro:Link reference="${prefix}link4_4"/>
+  <xacro:EndEffectorLink reference="${prefix}link5_4"/>
   <!-- Leg 5 links -->
   <xacro:Link reference="${prefix}link1_5"/>
@@ -51,4 +66,5 @@
   <xacro:Link reference="${prefix}link3_5"/>
   <xacro:Link reference="${prefix}link4_5"/>
+  <xacro:EndEffectorLink reference="${prefix}link5_5"/>
   <!-- Leg 6 links -->
   <xacro:Link reference="${prefix}link1_6"/>
@@ -56,4 +72,5 @@
   <xacro:Link reference="${prefix}link3_6"/>
   <xacro:Link reference="${prefix}link4_6"/>
+  <xacro:EndEffectorLink reference="${prefix}link5_6"/>
   <!-- Leg 1 Transmissions -->
   <xacro:SimpleTransmission trans="${prefix}leg1_trans1" joint="${prefix}joint1_1" actuator="${prefix}leg1_motor1" />

File: sim_and_real/ros2_ws_hex/src/hexapod_description/urdf/hexapod_ee.urdf.xacro (robot description, xacro)
@@ -9,5 +9,5 @@
     <xacro:hexapod_leg_ee prefix="${prefix}" version="${version}"/>
     <xacro:hexapod_gazebo prefix="${prefix}" />
-    <xacro:imu_sensor
+    <!-- <xacro:imu_sensor
     prefix="${prefix}"
     parent="${prefix}base_link"
@@ -16,5 +16,5 @@
     rpy_offset="0 0 0"
     update_rate="15.0"
-    topic_name="imu/data"/>
+    topic_name="imu/data"/> -->
     <gazebo>
       <plugin filename="gz_ros2_control-system" name="gz_ros2_control::GazeboSimROS2ControlPlugin">
@@ -22,16 +22,10 @@
       </plugin>
     </gazebo>
-    <gazebo reference="imu">
+    <gazebo reference="${prefix}base_link">
       <sensor name="imu_sensor" type="imu">
-        <update_rate>100.0</update_rate>
+        <update_rate>1</update_rate>
         <always_on>true</always_on>
-        <visualize>true</visualize>
-        <topic>imu/data</topic>
-        <imu>
-          <topic>imu/data</topic>
-          <gaussian_noise>0.01</gaussian_noise>
-          <bias_mean>0.0</bias_mean>
-          <bias_stddev>0.0</bias_stddev>
-        </imu>
+        <visualize>false</visualize>
+        <topic>imu</topic>
       </sensor>
     </gazebo>

Commit message: add contact sensors for each leg

File: sim_and_real/ros2_ws_hex/src/hexapod_description/gazebo/hexapod.gazebo.xacro (robot description, xacro)
@@ -25,5 +25,5 @@
   </xacro:macro>
   <!-- Gazebo reference for end effector link -->
-   <xacro:macro name="EndEffectorLink" params="reference">
+   <xacro:macro name="EndEffectorLink" params="reference index">
     <gazebo reference="${reference}">
       <kp>1000000.0</kp>
@@ -34,5 +34,19 @@
       <minDepth>0.001</minDepth>
     </gazebo>
+    <gazebo reference="${prefix}link5_${index}">
+      <sensor name='sensor_contact_${index}' type='contact'>
+          <contact>
+              <collision>link5_${index}_collision</collision>
+          </contact>
+      </sensor>
+    </gazebo>
    </xacro:macro>
+    <!-- <gazebo reference="${prefix}link5_3">
+      <sensor name='sensor_contact_3' type='contact'>
+          <contact>
+              <collision>link5_3_collision</collision>
+          </contact>
+      </sensor>
+    </gazebo> -->
   <!-- Define links for all parts of the hexapod -->
   <xacro:Link reference="${prefix}base_link"/>
@@ -42,5 +56,5 @@
   <xacro:Link reference="${prefix}link3_1"/>
   <xacro:Link reference="${prefix}link4_1"/>
-  <xacro:EndEffectorLink reference="${prefix}link5_1"/>
+  <xacro:EndEffectorLink reference="${prefix}link5_1" index="1"/>
   <!-- Leg 2 links -->
   <xacro:Link reference="${prefix}link1_2"/>
@@ -48,5 +62,5 @@
   <xacro:Link reference="${prefix}link3_2"/>
   <xacro:Link reference="${prefix}link4_2"/>
-  <xacro:EndEffectorLink reference="${prefix}link5_2"/>
+  <xacro:EndEffectorLink reference="${prefix}link5_2" index="2"/>
   <!-- Leg 3 links -->
   <xacro:Link reference="${prefix}link1_3"/>
@@ -54,5 +68,5 @@
   <xacro:Link reference="${prefix}link3_3"/>
   <xacro:Link reference="${prefix}link4_3"/>
-  <xacro:EndEffectorLink reference="${prefix}link5_3"/>
+  <xacro:EndEffectorLink reference="${prefix}link5_3" index="3"/>
   <!-- Leg 4 links -->
   <xacro:Link reference="${prefix}link1_4"/>
@@ -60,5 +74,5 @@
   <xacro:Link reference="${prefix}link3_4"/>
   <xacro:Link reference="${prefix}link4_4"/>
-  <xacro:EndEffectorLink reference="${prefix}link5_4"/>
+  <xacro:EndEffectorLink reference="${prefix}link5_4" index="4"/>
   <!-- Leg 5 links -->
   <xacro:Link reference="${prefix}link1_5"/>
@@ -66,5 +80,5 @@
   <xacro:Link reference="${prefix}link3_5"/>
   <xacro:Link reference="${prefix}link4_5"/>
-  <xacro:EndEffectorLink reference="${prefix}link5_5"/>
+  <xacro:EndEffectorLink reference="${prefix}link5_5" index="5"/>
   <!-- Leg 6 links -->
   <xacro:Link reference="${prefix}link1_6"/>
@@ -72,5 +86,5 @@
   <xacro:Link reference="${prefix}link3_6"/>
   <xacro:Link reference="${prefix}link4_6"/>
-  <xacro:EndEffectorLink reference="${prefix}link5_6"/>
+  <xacro:EndEffectorLink reference="${prefix}link5_6" index="6"/>
   <!-- Leg 1 Transmissions -->
   <xacro:SimpleTransmission trans="${prefix}leg1_trans1" joint="${prefix}joint1_1" actuator="${prefix}leg1_motor1" />

File: sim_and_real/ros2_ws_hex/src/hexapod_description/urdf/hexapod_ee.urdf.xacro (robot description, xacro)
@@ -4,5 +4,5 @@
     <xacro:include filename="$(find hexapod_description)/gazebo/hexapod.gazebo.xacro" />
     <xacro:include filename="$(find hexapod_description)/urdf/hexapod_leg_ee.urdf.xacro" />
-    <xacro:include filename="$(find hexapod_description)/urdf/hexapod_gazebo.urdf.xacro" />
+    <!-- <xacro:include filename="$(find hexapod_description)/urdf/hexapod_gazebo.urdf.xacro" /> -->
     <xacro:include filename="$(find hexapod_description)/urdf/imu.urdf.xacro"/>
     <xacro:include filename="$(find hexapod_moveit_config)/config/hexapod.ros2_control.xacro" />
@@ -31,11 +31,4 @@
       </plugin>
     </gazebo>
-    <gazebo reference="${prefix}link5_1">
-      <sensor name='sensor_contact_1' type='contact'>
-          <contact>
-              <collision>link5_1_collision</collision>
-          </contact>
-      </sensor>
-    </gazebo>
     <gazebo reference="${prefix}base_link">
       <sensor name="imu_sensor" type="imu">

Commit message: Fixed moveit motion planning error

File: sim_and_real/ros2_ws_hex/src/hexapod_description/gazebo/hexapod.gazebo.xacro (robot description, xacro)
@@ -34,19 +34,13 @@
       <minDepth>0.001</minDepth>
     </gazebo>
-    <gazebo reference="${prefix}link5_${index}">
+    <gazebo reference="${prefix}link4_${index}">
       <sensor name='sensor_contact_${index}' type='contact'>
           <contact>
-              <collision>link5_${index}_collision</collision>
+              <!-- <collision>link5_${index}_collision</collision> -->
+               <collision>link4_${index}_fixed_joint_lump__link5_${index}_collision_4</collision>
           </contact>
       </sensor>
     </gazebo>
    </xacro:macro>
-    <!-- <gazebo reference="${prefix}link5_3">
-      <sensor name='sensor_contact_3' type='contact'>
-          <contact>
-              <collision>link5_3_collision</collision>
-          </contact>
-      </sensor>
-    </gazebo> -->
   <!-- Define links for all parts of the hexapod -->
   <xacro:Link reference="${prefix}base_link"/>
@@ -55,36 +49,36 @@
   <xacro:Link reference="${prefix}link2_1"/>
   <xacro:Link reference="${prefix}link3_1"/>
-  <xacro:Link reference="${prefix}link4_1"/>
-  <xacro:EndEffectorLink reference="${prefix}link5_1" index="1"/>
+  <!-- <xacro:Link reference="${prefix}link4_1"/> -->
+  <xacro:EndEffectorLink reference="${prefix}link4_1" index="1"/>
   <!-- Leg 2 links -->
   <xacro:Link reference="${prefix}link1_2"/>
   <xacro:Link reference="${prefix}link2_2"/>
   <xacro:Link reference="${prefix}link3_2"/>
-  <xacro:Link reference="${prefix}link4_2"/>
-  <xacro:EndEffectorLink reference="${prefix}link5_2" index="2"/>
+  <!-- <xacro:Link reference="${prefix}link4_2"/> -->
+  <xacro:EndEffectorLink reference="${prefix}link4_2" index="2"/>
   <!-- Leg 3 links -->
   <xacro:Link reference="${prefix}link1_3"/>
   <xacro:Link reference="${prefix}link2_3"/>
   <xacro:Link reference="${prefix}link3_3"/>
-  <xacro:Link reference="${prefix}link4_3"/>
-  <xacro:EndEffectorLink reference="${prefix}link5_3" index="3"/>
+  <!-- <xacro:Link reference="${prefix}link4_3"/> -->
+  <xacro:EndEffectorLink reference="${prefix}link4_3" index="3"/>
   <!-- Leg 4 links -->
   <xacro:Link reference="${prefix}link1_4"/>
   <xacro:Link reference="${prefix}link2_4"/>
   <xacro:Link reference="${prefix}link3_4"/>
-  <xacro:Link reference="${prefix}link4_4"/>
-  <xacro:EndEffectorLink reference="${prefix}link5_4" index="4"/>
+  <!-- <xacro:Link reference="${prefix}link4_4"/> -->
+  <xacro:EndEffectorLink reference="${prefix}link4_4" index="4"/>
   <!-- Leg 5 links -->
   <xacro:Link reference="${prefix}link1_5"/>
   <xacro:Link reference="${prefix}link2_5"/>
   <xacro:Link reference="${prefix}link3_5"/>
-  <xacro:Link reference="${prefix}link4_5"/>
-  <xacro:EndEffectorLink reference="${prefix}link5_5" index="5"/>
+  <!-- <xacro:Link reference="${prefix}link4_5"/> -->
+  <xacro:EndEffectorLink reference="${prefix}link4_5" index="5"/>
   <!-- Leg 6 links -->
   <xacro:Link reference="${prefix}link1_6"/>
   <xacro:Link reference="${prefix}link2_6"/>
   <xacro:Link reference="${prefix}link3_6"/>
-  <xacro:Link reference="${prefix}link4_6"/>
-  <xacro:EndEffectorLink reference="${prefix}link5_6" index="6"/>
+  <!-- <xacro:Link reference="${prefix}link4_6"/> -->
+  <xacro:EndEffectorLink reference="${prefix}link4_6" index="6"/>
   <!-- Leg 1 Transmissions -->
   <xacro:SimpleTransmission trans="${prefix}leg1_trans1" joint="${prefix}joint1_1" actuator="${prefix}leg1_motor1" />

File: sim_and_real/ros2_ws_hex/src/hexapod_description/urdf/hexapod_leg_ee.urdf.xacro (robot description, xacro)
@@ -370,9 +370,9 @@
   <!-- Macro: Effector Joint -->
   <xacro:macro name="end_effector_joint" params="prefix index xyz rpy">
-    <joint name="${prefix}joint4_${index}" type="revolute">
+    <joint name="${prefix}joint4_${index}" type="fixed">
       <parent link="${prefix}link4_${index}"/>
       <child link="${prefix}link5_${index}"/>
       <origin xyz="${xyz}" rpy="${rpy}"/>
-      <limit effort="5.0" velocity="1.0" lower="0" upper="0"/>
+      <!-- <limit effort="5.0" velocity="1.0" lower="0" upper="0"/> -->
     </joint>
   </xacro:macro>

File: sim_and_real/ros2_ws_hex/src/hexapod_moveit_config/config/hexapod.ros2_control.xacro (robot description, xacro)
@@ -52,8 +52,8 @@
                 <state_interface name="velocity"/>
             </joint>
-            <joint name="joint4_1">
+            <!-- <joint name="joint4_1">
                 <command_interface name="position"/>
                 <state_interface name="position"/>
-            </joint>
+            </joint> -->
             <!-- Leg 2 joints -->
             <joint name="joint1_2">
@@ -78,8 +78,8 @@
                 <state_interface name="velocity"/>
             </joint>
-            <joint name="joint4_2">
+            <!-- <joint name="joint4_2">
                 <command_interface name="position"/>
                 <state_interface name="position"/>
-            </joint>
+            </joint> -->
             <!-- Leg 3 joints -->
             <joint name="joint1_3">
@@ -104,8 +104,8 @@
                 <state_interface name="velocity"/>
             </joint>
-            <joint name="joint4_3">
+            <!-- <joint name="joint4_3">
                 <command_interface name="position"/>
                 <state_interface name="position"/>
-            </joint>
+            </joint> -->
             <!-- Leg 4 joints -->
             <joint name="joint1_4">
@@ -130,8 +130,8 @@
                 <state_interface name="velocity"/>
             </joint>
-            <joint name="joint4_4">
+            <!-- <joint name="joint4_4">
                 <command_interface name="position"/>
                 <state_interface name="position"/>
-            </joint>
+            </joint> -->
             <!-- Leg 5 joints -->
             <joint name="joint1_5">
@@ -156,8 +156,8 @@
                 <state_interface name="velocity"/>
             </joint>
-            <joint name="joint4_5">
+            <!-- <joint name="joint4_5">
                 <command_interface name="position"/>
                 <state_interface name="position"/>
-            </joint>
+            </joint> -->
             <!-- Leg 6 joints -->
             <joint name="joint1_6">
@@ -182,8 +182,8 @@
                 <state_interface name="velocity"/>
             </joint>
-            <joint name="joint4_6">
+            <!-- <joint name="joint4_6">
                 <command_interface name="position"/>
                 <state_interface name="position"/>
-            </joint>
+            </joint> -->
         </ros2_control>
     </xacro:macro>
