Commit message: I updated position of center of masses and collision model for platform

File: sim_and_real/ros2_ws_hex/src/hexapod_description/collision/Version2/down_section_hitbox.xacro (robot description, xacro)
@@ -15,42 +15,42 @@
         <!-- Define geometric shapes with their relative positions and sizes from CSV data -->
         <!-- Cube 0 -->
-        <xacro:property name="cube_0_size_x" value="0.07840"/>
-        <xacro:property name="cube_0_size_y" value="0.03920"/>
-        <xacro:property name="cube_0_size_z" value="0.02760"/>
-        <xacro:property name="cube_0_offset_x" value="-0.07438"/>
-        <xacro:property name="cube_0_offset_y" value="-0.00010"/>
-        <xacro:property name="cube_0_offset_z" value="0.00000"/>
-        <xacro:property name="cube_0_roll" value="0.00000"/>
-        <xacro:property name="cube_0_pitch" value="0.00000"/>
-        <xacro:property name="cube_0_yaw" value="0.00000"/>
+        <xacro:property name="cube_0_size_x" value="0.0784"/>
+        <xacro:property name="cube_0_size_y" value="0.0392"/>
+        <xacro:property name="cube_0_size_z" value="0.0276"/>
+        <xacro:property name="cube_0_offset_x" value="-0.047685"/>
+        <xacro:property name="cube_0_offset_y" value="0"/>
+        <xacro:property name="cube_0_offset_z" value="0.0001"/>
+        <xacro:property name="cube_0_roll" value="0"/>
+        <xacro:property name="cube_0_pitch" value="0"/>
+        <xacro:property name="cube_0_yaw" value="0"/>
         <!-- Cube 1 -->
-        <xacro:property name="cube_1_size_x" value="0.11400"/>
-        <xacro:property name="cube_1_size_y" value="0.02340"/>
-        <xacro:property name="cube_1_size_z" value="0.02720"/>
-        <xacro:property name="cube_1_offset_x" value="0.02064"/>
-        <xacro:property name="cube_1_offset_y" value="-0.00010"/>
-        <xacro:property name="cube_1_offset_z" value="0.00000"/>
-        <xacro:property name="cube_1_roll" value="0.00000"/>
-        <xacro:property name="cube_1_pitch" value="0.00000"/>
-        <xacro:property name="cube_1_yaw" value="0.00000"/>
+        <xacro:property name="cube_1_size_x" value="0.114"/>
+        <xacro:property name="cube_1_size_y" value="0.0234"/>
+        <xacro:property name="cube_1_size_z" value="0.0272"/>
+        <xacro:property name="cube_1_offset_x" value="0.047741"/>
+        <xacro:property name="cube_1_offset_y" value="-0.0001"/>
+        <xacro:property name="cube_1_offset_z" value="0.0007"/>
+        <xacro:property name="cube_1_roll" value="0"/>
+        <xacro:property name="cube_1_pitch" value="0"/>
+        <xacro:property name="cube_1_yaw" value="0"/>
         <!-- Cube 2 -->
-        <xacro:property name="cube_2_size_x" value="0.03520"/>
-        <xacro:property name="cube_2_size_y" value="0.01180"/>
-        <xacro:property name="cube_2_size_z" value="0.03780"/>
-        <xacro:property name="cube_2_offset_x" value="0.04692"/>
-        <xacro:property name="cube_2_offset_y" value="0.00000"/>
-        <xacro:property name="cube_2_offset_z" value="0.00000"/>
-        <xacro:property name="cube_2_roll" value="0.00000"/>
-        <xacro:property name="cube_2_pitch" value="0.00000"/>
-        <xacro:property name="cube_2_yaw" value="0.00000"/>
+        <xacro:property name="cube_2_size_x" value="0.0352"/>
+        <xacro:property name="cube_2_size_y" value="0.0118"/>
+        <xacro:property name="cube_2_size_z" value="0.0378"/>
+        <xacro:property name="cube_2_offset_x" value="0.0725"/>
+        <xacro:property name="cube_2_offset_y" value="0"/>
+        <xacro:property name="cube_2_offset_z" value="0"/>
+        <xacro:property name="cube_2_roll" value="0"/>
+        <xacro:property name="cube_2_pitch" value="0"/>
+        <xacro:property name="cube_2_yaw" value="0"/>
         <!-- Cylinder 0 -->
-        <xacro:property name="cylinder_0_radius" value="0.01850"/>
-        <xacro:property name="cylinder_0_length" value="0.03920"/>
-        <xacro:property name="cylinder_0_offset_x" value="-0.11702"/>
-        <xacro:property name="cylinder_0_offset_y" value="-0.00005"/>
-        <xacro:property name="cylinder_0_offset_z" value="-0.00458"/>
-        <xacro:property name="cylinder_0_roll" value="1.57080"/>
-        <xacro:property name="cylinder_0_pitch" value="0.00000"/>
-        <xacro:property name="cylinder_0_yaw" value="0.00000"/>
+        <xacro:property name="cylinder_0_radius" value="0.00925"/>
+        <xacro:property name="cylinder_0_length" value="0.0392"/>
+        <xacro:property name="cylinder_0_offset_x" value="-0.0894"/>
+        <xacro:property name="cylinder_0_offset_y" value="-0.00005114"/>
+        <xacro:property name="cylinder_0_offset_z" value="-0.0042807"/>
+        <xacro:property name="cylinder_0_roll" value="1.570796327"/>
+        <xacro:property name="cylinder_0_pitch" value="0"/>
+        <xacro:property name="cylinder_0_yaw" value="0"/>
         <!-- Calculate rotation components for main rotation -->
         <xacro:property name="cr" value="${cos(roll)}"/>

File: sim_and_real/ros2_ws_hex/src/hexapod_description/collision/Version2/mid_section_hitbox.xacro (robot description, xacro)
@@ -18,7 +18,7 @@
         <xacro:property name="cube_0_size_y" value="0.039400"/>
         <xacro:property name="cube_0_size_z" value="0.062800"/>
-        <xacro:property name="cube_0_offset_x" value="0.004280"/>
-        <xacro:property name="cube_0_offset_y" value="0.000000"/>
-        <xacro:property name="cube_0_offset_z" value="0.007230"/>
+        <xacro:property name="cube_0_offset_x" value="-0.000123"/>
+        <xacro:property name="cube_0_offset_y" value="0.000023"/>
+        <xacro:property name="cube_0_offset_z" value="0.001713"/>
         <xacro:property name="cube_0_roll" value="0.000000"/>
         <xacro:property name="cube_0_pitch" value="0.000000"/>
@@ -26,8 +26,8 @@
         <!-- Cylinder 0 -->
         <xacro:property name="cylinder_0_radius" value="0.019300"/>
-        <xacro:property name="cylinder_0_length" value="0.020000"/>
-        <xacro:property name="cylinder_0_offset_x" value="-0.056378"/>
-        <xacro:property name="cylinder_0_offset_y" value="0.000000"/>
-        <xacro:property name="cylinder_0_offset_z" value="0.000000"/>
+        <xacro:property name="cylinder_0_length" value="0.040000"/>
+        <xacro:property name="cylinder_0_offset_x" value="-0.060781"/>
+        <xacro:property name="cylinder_0_offset_y" value="0.000023"/>
+        <xacro:property name="cylinder_0_offset_z" value="-0.005517"/>
         <xacro:property name="cylinder_0_roll" value="1.570796"/>
         <xacro:property name="cylinder_0_pitch" value="0.000000"/>
@@ -35,8 +35,8 @@
         <!-- Cylinder 1 -->
         <xacro:property name="cylinder_1_radius" value="0.019300"/>
-        <xacro:property name="cylinder_1_length" value="0.020000"/>
-        <xacro:property name="cylinder_1_offset_x" value="0.064572"/>
-        <xacro:property name="cylinder_1_offset_y" value="0.000000"/>
-        <xacro:property name="cylinder_1_offset_z" value="0.000000"/>
+        <xacro:property name="cylinder_1_length" value="0.040000"/>
+        <xacro:property name="cylinder_1_offset_x" value="0.060169"/>
+        <xacro:property name="cylinder_1_offset_y" value="0.000023"/>
+        <xacro:property name="cylinder_1_offset_z" value="-0.005517"/>
         <xacro:property name="cylinder_1_roll" value="1.570796"/>
         <xacro:property name="cylinder_1_pitch" value="0.000000"/>

File: sim_and_real/ros2_ws_hex/src/hexapod_description/collision/Version2/platform_hitbox.xacro (robot description, xacro)
@@ -5,47 +5,47 @@
     <!-- Sześcian 0 -->
     <collision>
-      <origin xyz="0 0 0.00210" rpy="0 0 0"/>
+      <origin xyz="0 0 0.0161" rpy="0.00000 0.00000 0.00000"/>
       <geometry>
-        <box size="0.19000 0.07820 0.00320"/>
+        <box size="0.07820 0.19000 0.0288"/>
       </geometry>
     </collision>
     <!-- Sześcian 1 -->
     <collision>
-      <origin xyz="0.04104 0.04082 0.00210" rpy="0 0 0.78540"/>
+      <origin xyz="0.04104 0.04082 0.0161" rpy="0.00000 0.00000 0.78540"/>
       <geometry>
-        <box size="0.07320 0.08000 0.00320"/>
+        <box size="0.07320 0.08000 0.0288"/>
       </geometry>
     </collision>
     <!-- Sześcian 2 -->
     <collision>
-      <origin xyz="0.04104 -0.04082 0.00210" rpy="0 0 -0.78540"/>
+      <origin xyz="0.04104 -0.04082 0.0161" rpy="0.00000 0.00000 -0.78540"/>
       <geometry>
-        <box size="0.07320 0.08000 0.00320"/>
+        <box size="0.07320 0.08000 0.0288"/>
       </geometry>
     </collision>
     <!-- Sześcian 3 -->
     <collision>
-      <origin xyz="-0.04104 0.04082 0.00210" rpy="0 0 -0.78540"/>
+      <origin xyz="-0.04104 0.04082 0.0161" rpy="0.00000 0.00000 -0.78540"/>
       <geometry>
-        <box size="0.07320 0.08000 0.00320"/>
+        <box size="0.07320 0.08000 0.0288"/>
       </geometry>
     </collision>
     <!-- Sześcian 4 -->
     <collision>
-      <origin xyz="-0.04104 -0.04082 0.00210" rpy="0 0 0.78540"/>
+      <origin xyz="-0.04104 -0.04082 0.0161" rpy="0.00000 0.00000 0.78540"/>
       <geometry>
-        <box size="0.07320 0.08000 0.00320"/>
+        <box size="0.07320 0.08000 0.0288"/>
       </geometry>
     </collision>
     <!-- Sześcian 5 -->
     <collision>
-      <origin xyz="0 0 0.00210" rpy="0 0 0"/>
+      <origin xyz="0 0 0.01556" rpy="0.00000 0.00000 0.00000"/>
       <geometry>
-        <box size="0.07820 0.19000 0.00320"/>
+        <box size="0.07820 0.19000 0.0288"/>
       </geometry>
     </collision>
     <!-- Sześcian 6 -->
     <collision>
-      <origin xyz="-0.08452 0.00975 -0.00693" rpy="0 0 1.57080"/>
+      <origin xyz="-0.08452 0.00975 -0.00693" rpy="0.00000 0.00000 1.57080"/>
       <geometry>
         <box size="0.04060 0.02100 0.03880"/>
@@ -54,5 +54,5 @@
     <!-- Sześcian 7 -->
     <collision>
-      <origin xyz="-0.05269 0.06718 -0.00693" rpy="0 0 0.78540"/>
+      <origin xyz="-0.05269 0.06718 -0.00693" rpy="0.00000 0.00000 0.78540"/>
       <geometry>
         <box size="0.04060 0.02100 0.03880"/>
@@ -61,5 +61,5 @@
     <!-- Sześcian 8 -->
     <collision>
-      <origin xyz="0.05269 0.06718 -0.00693" rpy="0 0 -0.78540"/>
+      <origin xyz="0.05269 0.06718 -0.00693" rpy="0.00000 0.00000 -0.78540"/>
       <geometry>
         <box size="0.04060 0.02100 0.03880"/>
@@ -68,5 +68,5 @@
     <!-- Sześcian 9 -->
     <collision>
-      <origin xyz="-0.06759 -0.05244 -0.00693" rpy="0 0 -0.78540"/>
+      <origin xyz="-0.06759 -0.05244 -0.00693" rpy="0.00000 0.00000 -0.78540"/>
       <geometry>
         <box size="0.04060 0.02100 0.03880"/>
@@ -75,5 +75,5 @@
     <!-- Sześcian 10 -->
     <collision>
-      <origin xyz="0.06759 -0.05244 -0.00693" rpy="0 0 0.78540"/>
+      <origin xyz="0.06759 -0.05244 -0.00693" rpy="0.00000 0.00000 0.78540"/>
       <geometry>
         <box size="0.04060 0.02100 0.03880"/>
@@ -82,49 +82,98 @@
     <!-- Sześcian 11 -->
     <collision>
-      <origin xyz="0.08452 0.00975 -0.00693" rpy="0 0 1.57080"/>
+      <origin xyz="0.08452 0.00975 -0.00693" rpy="0.00000 0.00000 1.57080"/>
       <geometry>
         <box size="0.04060 0.02100 0.03880"/>
       </geometry>
     </collision>
+    <!-- Sześcian 12 -->
+    <collision>
+      <origin xyz="0 0 0.0161" rpy="0.00000 0.00000 1.57080"/>
+      <geometry>
+        <box size="0.07820 0.19000 0.0288"/>
+      </geometry>
+    </collision>
+    <!-- Sześcian 13 -->
+    <collision>
+      <origin xyz="-0.07305 -0.06865 0.0161" rpy="0.00000 0.00000 0.7853981634"/>
+      <geometry>
+        <box size="0.0502 0.0724 0.0344"/>
+      </geometry>
+    </collision>
+    <!-- Sześcian 14 -->
+    <collision>
+      <origin xyz="-0.06843 0.07413 0.0161" rpy="0.00000 0.00000 -0.7853981634"/>
+      <geometry>
+        <box size="0.0502 0.0758 0.0344"/>
+      </geometry>
+    </collision>
+    <!-- Sześcian 15 -->
+    <collision>
+      <origin xyz="0.06843 0.07413 0.0161" rpy="0.00000 0.00000 3.926990817"/>
+      <geometry>
+        <box size="0.0502 0.0758 0.0344"/>
+      </geometry>
+    </collision>
+    <!-- Sześcian 16 -->
+    <collision>
+      <origin xyz="0.09828 0.0053 0.0161" rpy="0.00000 0.00000 1.570796327"/>
+      <geometry>
+        <box size="0.0772 0.0536 0.0344"/>
+      </geometry>
+    </collision>
+    <!-- Sześcian 17 -->
+    <collision>
+      <origin xyz="-0.09828 0.0053 0.0161" rpy="0.00000 0.00000 1.570796327"/>
+      <geometry>
+        <box size="0.0772 0.0536 0.0344"/>
+      </geometry>
+    </collision>
+    <!-- Sześcian 18 -->
+    <collision>
+      <origin xyz="0.07305 -0.06865 0.0161" rpy="0.00000 0.00000 2.35619449"/>
+      <geometry>
+        <box size="0.0772 0.0536 0.0344"/>
+      </geometry>
+    </collision>
     <!-- Cylinder 0 -->
     <collision>
-      <origin xyz="0.08573 0 0.01696" rpy="0 0 0"/>
+      <origin xyz="0.08600 -0.08607 0.01708" rpy="0.00000 0.00000 0.00000"/>
       <geometry>
-        <cylinder radius="0.014" length="0.00840"/>
+        <cylinder radius="0.014" length="0.0278"/>
       </geometry>
     </collision>
     <!-- Cylinder 1 -->
     <collision>
-      <origin xyz="-0.08573 0 0.01696" rpy="0 0 0"/>
+      <origin xyz="-0.08600 -0.08607 0.01708" rpy="0.00000 0.00000 0.00000"/>
       <geometry>
-        <cylinder radius="0.014" length="0.00840"/>
+        <cylinder radius="0.014" length="0.0278"/>
       </geometry>
     </collision>
     <!-- Cylinder 2 -->
     <collision>
-      <origin xyz="-0.06054 -0.06009 0.01696" rpy="0 0 0"/>
+      <origin xyz="0.08600 0.08607 0.01708" rpy="0.00000 0.00000 0.00000"/>
       <geometry>
-        <cylinder radius="0.014" length="0.00840"/>
+        <cylinder radius="0.014" length="0.0278"/>
       </geometry>
     </collision>
     <!-- Cylinder 3 -->
     <collision>
-      <origin xyz="-0.06054 0.06009 0.01696" rpy="0 0 0"/>
+      <origin xyz="-0.08600 0.08607 0.01708" rpy="0.00000 0.00000 0.00000"/>
       <geometry>
-        <cylinder radius="0.014" length="0.00840"/>
+        <cylinder radius="0.014" length="0.0278"/>
       </geometry>
     </collision>
     <!-- Cylinder 4 -->
     <collision>
-      <origin xyz="0.06054 -0.06009 0.01696" rpy="0 0 0"/>
+      <origin xyz="0.12206 0.00017 0.01708" rpy="0.00000 0.00000 0.00000"/>
       <geometry>
-        <cylinder radius="0.014" length="0.00840"/>
+        <cylinder radius="0.014" length="0.0278"/>
       </geometry>
     </collision>
     <!-- Cylinder 5 -->
     <collision>
-      <origin xyz="0.06054 0.06009 0.01696" rpy="0 0 0"/>
+      <origin xyz="-0.12206 0.00017 0.01708" rpy="0.00000 0.00000 0.00000"/>
       <geometry>
-        <cylinder radius="0.014" length="0.00840"/>
+        <cylinder radius="0.014" length="0.0278"/>
       </geometry>
     </collision>

File: sim_and_real/ros2_ws_hex/src/hexapod_description/collision/Version2/tip_hitbox.xacro (robot description, xacro)
@@ -16,5 +16,5 @@
         <xacro:property name="sphere_0_radius" value="0.00600"/>
         <!-- <xacro:property name="sphere_0_offset_x" value="0.00000"/> ORYGINALNA WARTOŚĆ -->
-        <xacro:property name="sphere_0_offset_x" value="-0.00500"/> <!--TUTAJ ZMNIEJSZAMY [M] ABY DODAĆ PRZESUNIĘCIE SYMULUJĄCE ODGIĘCIE SPRĘŻYNY -->
+        <xacro:property name="sphere_0_offset_x" value="-0.0025"/> <!--TUTAJ ZMNIEJSZAMY [M] ABY DODAĆ PRZESUNIĘCIE SYMULUJĄCE ODGIĘCIE SPRĘŻYNY -->
         <xacro:property name="sphere_0_offset_y" value="0.00000"/> <!--NA RAZIE JEST 0.5CM -->
         <xacro:property name="sphere_0_offset_z" value="0.00000"/>
@@ -26,5 +26,5 @@
         <xacro:property name="cylinder_0_length" value="0.01080"/>
         <!-- <xacro:property name="cylinder_0_offset_x" value="-0.00918"/> ORYGINALNA WARTOŚĆ -->
-        <xacro:property name="cylinder_0_offset_x" value="-0.01418"/> <!--TUTAJ ZMNIEJSZAMY [M] ABY DODAĆ PRZESUNIĘCIE SYMULUJĄCE ODGIĘCIE SPRĘŻYNY -->
+        <xacro:property name="cylinder_0_offset_x" value="-0.00918"/> <!--TUTAJ ZMNIEJSZAMY [M] ABY DODAĆ PRZESUNIĘCIE SYMULUJĄCE ODGIĘCIE SPRĘŻYNY -->
         <xacro:property name="cylinder_0_offset_y" value="0.00000"/>
         <xacro:property name="cylinder_0_offset_z" value="0.00031"/>

File: sim_and_real/ros2_ws_hex/src/hexapod_description/collision/Version2/up_section_hitbox.xacro (robot description, xacro)
@@ -13,12 +13,12 @@
         <xacro:property name="pitch" value="${rot_parts[1]}"/>
         <xacro:property name="yaw" value="${rot_parts[2]}"/>
-        <!-- Define geometric shapes with their relative positions and sizes from CSV data V2 -->
+        <!-- Define geometric shapes with their relative positions and sizes from CSV data -->
         <!-- Cube 0 -->
         <xacro:property name="cube_0_size_x" value="0.022"/>
         <xacro:property name="cube_0_size_y" value="0.0316"/>
         <xacro:property name="cube_0_size_z" value="0.0282"/>
-        <xacro:property name="cube_0_offset_x" value="0.02212"/>
-        <xacro:property name="cube_0_offset_y" value="-0.00087"/>
-        <xacro:property name="cube_0_offset_z" value="0.00000"/>
+        <xacro:property name="cube_0_offset_x" value="0.00682"/>
+        <xacro:property name="cube_0_offset_y" value="-0.00061"/>
+        <xacro:property name="cube_0_offset_z" value="-0.00009"/>
         <xacro:property name="cube_0_roll" value="0.00000"/>
         <xacro:property name="cube_0_pitch" value="0.00000"/>
@@ -28,7 +28,7 @@
         <xacro:property name="cube_1_size_y" value="0.004"/>
         <xacro:property name="cube_1_size_z" value="0.036"/>
-        <xacro:property name="cube_1_offset_x" value="0.03631"/>
-        <xacro:property name="cube_1_offset_y" value="-0.01793"/>
-        <xacro:property name="cube_1_offset_z" value="0.00000"/>
+        <xacro:property name="cube_1_offset_x" value="0.02101"/>
+        <xacro:property name="cube_1_offset_y" value="-0.01767"/>
+        <xacro:property name="cube_1_offset_z" value="-0.00009"/>
         <xacro:property name="cube_1_roll" value="0.00000"/>
         <xacro:property name="cube_1_pitch" value="0.00000"/>
@@ -38,7 +38,7 @@
         <xacro:property name="cube_2_size_y" value="0.004"/>
         <xacro:property name="cube_2_size_z" value="0.036"/>
-        <xacro:property name="cube_2_offset_x" value="0.03631"/>
-        <xacro:property name="cube_2_offset_y" value="0.01793"/>
-        <xacro:property name="cube_2_offset_z" value="0.00000"/>
+        <xacro:property name="cube_2_offset_x" value="0.02101"/>
+        <xacro:property name="cube_2_offset_y" value="0.01819"/>
+        <xacro:property name="cube_2_offset_z" value="-0.00009"/>
         <xacro:property name="cube_2_roll" value="0.00000"/>
         <xacro:property name="cube_2_pitch" value="0.00000"/>
@@ -47,7 +47,7 @@
         <xacro:property name="cylinder_0_radius" value="0.014"/>
         <xacro:property name="cylinder_0_length" value="0.0306"/>
-        <xacro:property name="cylinder_0_offset_x" value="-0.00401"/>
-        <xacro:property name="cylinder_0_offset_y" value="-0.00012"/>
-        <xacro:property name="cylinder_0_offset_z" value="0.00000"/>
+        <xacro:property name="cylinder_0_offset_x" value="-0.01931"/>
+        <xacro:property name="cylinder_0_offset_y" value="0.00014"/>
+        <xacro:property name="cylinder_0_offset_z" value="-0.00009"/>
         <xacro:property name="cylinder_0_roll" value="0.00000"/>
         <xacro:property name="cylinder_0_pitch" value="0.00000"/>
@@ -56,7 +56,7 @@
         <xacro:property name="cylinder_1_radius" value="0.026"/>
         <xacro:property name="cylinder_1_length" value="0.0082"/>
-        <xacro:property name="cylinder_1_offset_x" value="-0.00400"/>
-        <xacro:property name="cylinder_1_offset_y" value="0.00000"/>
-        <xacro:property name="cylinder_1_offset_z" value="0.00000"/>
+        <xacro:property name="cylinder_1_offset_x" value="-0.01930"/>
+        <xacro:property name="cylinder_1_offset_y" value="0.00026"/>
+        <xacro:property name="cylinder_1_offset_z" value="-0.00009"/>
         <xacro:property name="cylinder_1_roll" value="0.00000"/>
         <xacro:property name="cylinder_1_pitch" value="0.00000"/>
@@ -65,7 +65,7 @@
         <xacro:property name="cylinder_2_radius" value="0.018"/>
         <xacro:property name="cylinder_2_length" value="0.004"/>
-        <xacro:property name="cylinder_2_offset_x" value="0.05482"/>
-        <xacro:property name="cylinder_2_offset_y" value="-0.01793"/>
-        <xacro:property name="cylinder_2_offset_z" value="0.00027"/>
+        <xacro:property name="cylinder_2_offset_x" value="0.03952"/>
+        <xacro:property name="cylinder_2_offset_y" value="-0.01767"/>
+        <xacro:property name="cylinder_2_offset_z" value="0.00017"/>
         <xacro:property name="cylinder_2_roll" value="1.57080"/>
         <xacro:property name="cylinder_2_pitch" value="0.00000"/>
@@ -74,7 +74,7 @@
         <xacro:property name="cylinder_3_radius" value="0.018"/>
         <xacro:property name="cylinder_3_length" value="0.004"/>
-        <xacro:property name="cylinder_3_offset_x" value="0.05482"/>
-        <xacro:property name="cylinder_3_offset_y" value="0.01793"/>
-        <xacro:property name="cylinder_3_offset_z" value="0.00027"/>
+        <xacro:property name="cylinder_3_offset_x" value="0.03952"/>
+        <xacro:property name="cylinder_3_offset_y" value="0.01819"/>
+        <xacro:property name="cylinder_3_offset_z" value="0.00017"/>
         <xacro:property name="cylinder_3_roll" value="1.57080"/>
         <xacro:property name="cylinder_3_pitch" value="0.00000"/>
