Commit message: Even more precise inertia. Fixed problem with wrong tip collision of leg 2. Updated friction coefficients

File: sim_and_real/ros2_ws_hex/src/hexapod_description/collision/Version2/down_section_hitbox.xacro (robot description, xacro)
@@ -28,5 +28,5 @@
         <xacro:property name="cube_1_size_y" value="0.0234"/>
         <xacro:property name="cube_1_size_z" value="0.0272"/>
-        <xacro:property name="cube_1_offset_x" value="0.047741"/>
+        <xacro:property name="cube_1_offset_x" value="0.0404408"/>
         <xacro:property name="cube_1_offset_y" value="-0.0001"/>
         <xacro:property name="cube_1_offset_z" value="0.0007"/>

File: sim_and_real/ros2_ws_hex/src/hexapod_description/gazebo/hexapod.gazebo.xacro (robot description, xacro)
@@ -18,6 +18,6 @@
       <kp>1000000.0</kp>
       <kd>100.0</kd>
-      <mu1>30.0</mu1>
-      <mu2>30.0</mu2>
+      <mu1>0.7</mu1>
+      <mu2>0.7</mu2>
       <maxVel>1.0</maxVel>
       <minDepth>0.001</minDepth>
@@ -29,6 +29,6 @@
       <kp>1000000.0</kp>
       <kd>100.0</kd>
-      <mu1>30.0</mu1>
-      <mu2>30.0</mu2>
+      <mu1>0.7</mu1>
+      <mu2>0.7</mu2>
       <maxVel>1.0</maxVel>
       <minDepth>0.001</minDepth>

File: sim_and_real/ros2_ws_hex/src/hexapod_description/urdf/hexapod_leg_ee.urdf.xacro (robot description, xacro)
@@ -38,5 +38,5 @@
       <xacro:property name="joint3_2_xyz" value="0.0 0.089946 0.00505"/>
       <xacro:property name="joint3_2_axis" value="-1 0 0"/>
-      <xacro:property name="joint4_2_xyz" value="0.000147 0.164223 -0.000046"/>
+      <xacro:property name="joint4_2_xyz" value="0.000051 0.164207 0.000046"/>
       <xacro:property name="joint4_2_axis" value="0 0 0"/>
       <!-- CECHY POŁOŻENIA LINKÓW LEG 2 -->
@@ -113,5 +113,5 @@
     </xacro:if>
     <!-- DLA NOWEJ WERSJI HEXAPODA ZMIENIĆ PONIŻSZE PARAMETRY -->
-    <xacro:if value="${int(version) == 2}">
+<xacro:if value="${int(version) == 2}">
       <!-- CECHY INERCJI -->
       <xacro:property name="platform_mass" value="0.8095" />
@@ -136,10 +136,10 @@
       <xacro:property name="joint3_velocity" value="4.1"/>
       <!-- CECHY INERCJI PLATFORMY -->
-      <xacro:property name="platform_ixx" value="0.002679580768"/>
-      <xacro:property name="platform_ixy" value="0.000000022139"/>
-      <xacro:property name="platform_ixz" value="-0.000000074882"/>
-      <xacro:property name="platform_iyy" value="0.004389472777"/>
-      <xacro:property name="platform_iyz" value="0.000027268278"/>
-      <xacro:property name="platform_izz" value="0.0066010831"/>
+      <xacro:property name="platform_ixx" value="2.782630e-03"/>
+      <xacro:property name="platform_ixy" value="3.151174e-07"/>
+      <xacro:property name="platform_ixz" value="-3.746570e-07"/>
+      <xacro:property name="platform_iyy" value="3.491645e-03"/>
+      <xacro:property name="platform_iyz" value="8.425825e-06"/>
+      <xacro:property name="platform_izz" value="5.824094e-03"/>
       <!-- CECHY INERCJI DLA KOŃCÓWKI -->
       <xacro:property name="tip_ixx" value="0.0000000144"/>
@@ -168,22 +168,22 @@
       <xacro:property name="link_tip_1_rpy" value="0 0 0.785398163"/>
       <!-- CECHY INERCJI LINKÓW LEG 1 -->
-      <xacro:property name="upper_leg_1_ixx" value="0.000028881"/>
-      <xacro:property name="upper_leg_1_ixy" value="-0.000015979"/>
-      <xacro:property name="upper_leg_1_ixz" value="0"/>
-      <xacro:property name="upper_leg_1_iyy" value="0.000028881"/>
-      <xacro:property name="upper_leg_1_iyz" value="0"/>
-      <xacro:property name="upper_leg_1_izz" value="0.000047692"/>
-      <xacro:property name="mid_leg_1_ixx" value="0.000206312"/>
-      <xacro:property name="mid_leg_1_ixy" value="-0.000142147"/>
-      <xacro:property name="mid_leg_1_ixz" value="0"/>
-      <xacro:property name="mid_leg_1_iyy" value="0.000206312"/>
-      <xacro:property name="mid_leg_1_iyz" value="0"/>
-      <xacro:property name="mid_leg_1_izz" value="0.000329761"/>
-      <xacro:property name="lower_leg_1_ixx" value="0.000176460"/>
-      <xacro:property name="lower_leg_1_ixy" value="-0.000161040"/>
-      <xacro:property name="lower_leg_1_ixz" value="0"/>
-      <xacro:property name="lower_leg_1_iyy" value="0.000176460"/>
-      <xacro:property name="lower_leg_1_iyz" value="0"/>
-      <xacro:property name="lower_leg_1_izz" value="0.000339420"/>
+      <xacro:property name="upper_leg_1_ixx" value="3.192059e-05"/>
+      <xacro:property name="upper_leg_1_ixy" value="-1.816964e-05"/>
+      <xacro:property name="upper_leg_1_ixz" value="-1.971549e-07"/>
+      <xacro:property name="upper_leg_1_iyy" value="3.172578e-05"/>
+      <xacro:property name="upper_leg_1_iyz" value="-6.665934e-08"/>
+      <xacro:property name="upper_leg_1_izz" value="5.413813e-05"/>
+      <xacro:property name="mid_leg_1_ixx" value="1.872470e-04"/>
+      <xacro:property name="mid_leg_1_ixy" value="-1.227141e-04"/>
+      <xacro:property name="mid_leg_1_ixz" value="4.021989e-08"/>
+      <xacro:property name="mid_leg_1_iyy" value="1.872811e-04"/>
+      <xacro:property name="mid_leg_1_iyz" value="7.655518e-08"/>
+      <xacro:property name="mid_leg_1_izz" value="2.854110e-04"/>
+      <xacro:property name="lower_leg_1_ixx" value="1.914881e-04"/>
+      <xacro:property name="lower_leg_1_ixy" value="-1.742340e-04"/>
+      <xacro:property name="lower_leg_1_ixz" value="-8.359193e-06"/>
+      <xacro:property name="lower_leg_1_iyy" value="1.914337e-04"/>
+      <xacro:property name="lower_leg_1_iyz" value="-8.346770e-06"/>
+      <xacro:property name="lower_leg_1_izz" value="3.656178e-04"/>
       <!-- CECHY POŁOŻENIA STAWÓW LEG 2 -->
       <xacro:property name="joint1_2_xyz" value="0.121845	0	0.0170504"/>
@@ -193,5 +193,5 @@
       <xacro:property name="joint3_2_xyz" value="0.120802	0.000000002	0"/>
       <xacro:property name="joint3_2_axis" value="0	1	0"/>
-      <xacro:property name="joint4_2_xyz" value="0.213498	-0.000094709	-0.004855"/>
+      <xacro:property name="joint4_2_xyz" value="0.213498	-0.000094709	0.004855"/>
       <xacro:property name="joint4_2_axis" value="0	0	0"/>
       <!-- CECHY POŁOŻENIA LINKÓW LEG 2 -->
@@ -206,22 +206,22 @@
       <xacro:property name="link_tip_2_rpy" value="0 0 0"/>
       <!-- CECHY INERCJI LINKÓW LEG 2 -->
-      <xacro:property name="upper_leg_2_ixx" value="0.000012901"/>
-      <xacro:property name="upper_leg_2_ixy" value="0"/>
-      <xacro:property name="upper_leg_2_ixz" value="0"/>
-      <xacro:property name="upper_leg_2_iyy" value="0.000044860"/>
-      <xacro:property name="upper_leg_2_iyz" value="0"/>
-      <xacro:property name="upper_leg_2_izz" value="0.000047692"/>
-      <xacro:property name="mid_leg_2_ixx" value="0.000064165"/>
-      <xacro:property name="mid_leg_2_ixy" value="0"/>
-      <xacro:property name="mid_leg_2_ixz" value="0"/>
-      <xacro:property name="mid_leg_2_iyy" value="0.000348459"/>
-      <xacro:property name="mid_leg_2_iyz" value="0"/>
-      <xacro:property name="mid_leg_2_izz" value="0.000329761"/>
-      <xacro:property name="lower_leg_2_ixx" value="0.000015420"/>
-      <xacro:property name="lower_leg_2_ixy" value="0"/>
-      <xacro:property name="lower_leg_2_ixz" value="0"/>
-      <xacro:property name="lower_leg_2_iyy" value="0.000337500"/>
-      <xacro:property name="lower_leg_2_iyz" value="0"/>
-      <xacro:property name="lower_leg_2_izz" value="0.000339420"/>
+      <xacro:property name="upper_leg_2_ixx" value="1.365355e-05"/>
+      <xacro:property name="upper_leg_2_ixy" value="-9.739604e-08"/>
+      <xacro:property name="upper_leg_2_ixz" value="-1.865458e-07"/>
+      <xacro:property name="upper_leg_2_iyy" value="4.999283e-05"/>
+      <xacro:property name="upper_leg_2_iyz" value="9.227452e-08"/>
+      <xacro:property name="upper_leg_2_izz" value="5.413814e-05"/>
+      <xacro:property name="mid_leg_2_ixx" value="6.454984e-05"/>
+      <xacro:property name="mid_leg_2_ixy" value="1.704929e-08"/>
+      <xacro:property name="mid_leg_2_ixz" value="8.257522e-08"/>
+      <xacro:property name="mid_leg_2_iyy" value="3.099780e-04"/>
+      <xacro:property name="mid_leg_2_iyz" value="2.569509e-08"/>
+      <xacro:property name="mid_leg_2_izz" value="2.854109e-04"/>
+      <xacro:property name="lower_leg_2_ixx" value="1.722692e-05"/>
+      <xacro:property name="lower_leg_2_ixy" value="-2.723387e-08"/>
+      <xacro:property name="lower_leg_2_ixz" value="-1.181289e-05"/>
+      <xacro:property name="lower_leg_2_iyy" value="3.656948e-04"/>
+      <xacro:property name="lower_leg_2_iyz" value="8.783736e-09"/>
+      <xacro:property name="lower_leg_2_izz" value="3.656178e-04"/>
       <!-- CECHY POŁOŻENIA STAWÓW LEG 3 -->
       <xacro:property name="joint1_3_xyz" value="0.0861847	-0.0860902	0.0170504"/>
@@ -244,22 +244,22 @@
       <xacro:property name="link_tip_3_rpy" value="0 0 5.497787144"/>
       <!-- CECHY INERCJI LINKÓW LEG 3 -->
-      <xacro:property name="upper_leg_3_ixx" value="0.000028881"/>
-      <xacro:property name="upper_leg_3_ixy" value="0.000015979"/>
-      <xacro:property name="upper_leg_3_ixz" value="0"/>
-      <xacro:property name="upper_leg_3_iyy" value="0.000028881"/>
-      <xacro:property name="upper_leg_3_iyz" value="0"/>
-      <xacro:property name="upper_leg_3_izz" value="0.000047692"/>
-      <xacro:property name="mid_leg_3_ixx" value="0.000206312"/>
-      <xacro:property name="mid_leg_3_ixy" value="0.000142147"/>
-      <xacro:property name="mid_leg_3_ixz" value="0"/>
-      <xacro:property name="mid_leg_3_iyy" value="0.000206312"/>
-      <xacro:property name="mid_leg_3_iyz" value="0"/>
-      <xacro:property name="mid_leg_3_izz" value="0.000329761"/>
-      <xacro:property name="lower_leg_3_ixx" value="0.000176460"/>
-      <xacro:property name="lower_leg_3_ixy" value="0.000161040"/>
-      <xacro:property name="lower_leg_3_ixz" value="0"/>
-      <xacro:property name="lower_leg_3_iyy" value="0.000176460"/>
-      <xacro:property name="lower_leg_3_iyz" value="0"/>
-      <xacro:property name="lower_leg_3_izz" value="0.000339420"/>
+      <xacro:property name="upper_leg_3_ixx" value="3.172580e-05"/>
+      <xacro:property name="upper_leg_3_ixy" value="1.816965e-05"/>
+      <xacro:property name="upper_leg_3_ixz" value="-6.666029e-08"/>
+      <xacro:property name="upper_leg_3_iyy" value="3.192058e-05"/>
+      <xacro:property name="upper_leg_3_iyz" value="1.971555e-07"/>
+      <xacro:property name="upper_leg_3_izz" value="5.413814e-05"/>
+      <xacro:property name="mid_leg_3_ixx" value="1.872811e-04"/>
+      <xacro:property name="mid_leg_3_ixy" value="1.227142e-04"/>
+      <xacro:property name="mid_leg_3_ixz" value="7.655505e-08"/>
+      <xacro:property name="mid_leg_3_iyy" value="1.872470e-04"/>
+      <xacro:property name="mid_leg_3_iyz" value="-4.021846e-08"/>
+      <xacro:property name="mid_leg_3_izz" value="2.854111e-04"/>
+      <xacro:property name="lower_leg_3_ixx" value="1.914336e-04"/>
+      <xacro:property name="lower_leg_3_ixy" value="1.742339e-04"/>
+      <xacro:property name="lower_leg_3_ixz" value="-8.346764e-06"/>
+      <xacro:property name="lower_leg_3_iyy" value="1.914880e-04"/>
+      <xacro:property name="lower_leg_3_iyz" value="8.359190e-06"/>
+      <xacro:property name="lower_leg_3_izz" value="3.656177e-04"/>
       <!-- CECHY POŁOŻENIA STAWÓW LEG 4 -->
       <xacro:property name="joint1_4_xyz" value="-0.0861847	-0.0860902	0.0170504"/>
@@ -282,22 +282,22 @@
       <xacro:property name="link_tip_4_rpy" value="0 0 3.926990817"/>
       <!-- CECHY INERCJI LINKÓW LEG 4 -->
-      <xacro:property name="upper_leg_4_ixx" value="0.000028881"/>
-      <xacro:property name="upper_leg_4_ixy" value="-0.000015979"/>
-      <xacro:property name="upper_leg_4_ixz" value="0"/>
-      <xacro:property name="upper_leg_4_iyy" value="0.000028881"/>
-      <xacro:property name="upper_leg_4_iyz" value="0"/>
-      <xacro:property name="upper_leg_4_izz" value="0.000047692"/>
-      <xacro:property name="mid_leg_4_ixx" value="0.000206312"/>
-      <xacro:property name="mid_leg_4_ixy" value="-0.000142147"/>
-      <xacro:property name="mid_leg_4_ixz" value="0"/>
-      <xacro:property name="mid_leg_4_iyy" value="0.000206312"/>
-      <xacro:property name="mid_leg_4_iyz" value="0"/>
-      <xacro:property name="mid_leg_4_izz" value="0.000329761"/>
-      <xacro:property name="lower_leg_4_ixx" value="0.000176460"/>
-      <xacro:property name="lower_leg_4_ixy" value="-0.000161040"/>
-      <xacro:property name="lower_leg_4_ixz" value="0"/>
-      <xacro:property name="lower_leg_4_iyy" value="0.000176460"/>
-      <xacro:property name="lower_leg_4_iyz" value="0"/>
-      <xacro:property name="lower_leg_4_izz" value="0.000339420"/>
+      <xacro:property name="upper_leg_4_ixx" value="3.192057e-05"/>
+      <xacro:property name="upper_leg_4_ixy" value="-1.816963e-05"/>
+      <xacro:property name="upper_leg_4_ixz" value="1.971549e-07"/>
+      <xacro:property name="upper_leg_4_iyy" value="3.172578e-05"/>
+      <xacro:property name="upper_leg_4_iyz" value="6.665899e-08"/>
+      <xacro:property name="upper_leg_4_izz" value="5.413811e-05"/>
+      <xacro:property name="mid_leg_4_ixx" value="1.872469e-04"/>
+      <xacro:property name="mid_leg_4_ixy" value="-1.227141e-04"/>
+      <xacro:property name="mid_leg_4_ixz" value="-4.021828e-08"/>
+      <xacro:property name="mid_leg_4_iyy" value="1.872811e-04"/>
+      <xacro:property name="mid_leg_4_iyz" value="-7.655551e-08"/>
+      <xacro:property name="mid_leg_4_izz" value="2.854110e-04"/>
+      <xacro:property name="lower_leg_4_ixx" value="1.914881e-04"/>
+      <xacro:property name="lower_leg_4_ixy" value="-1.742340e-04"/>
+      <xacro:property name="lower_leg_4_ixz" value="8.359195e-06"/>
+      <xacro:property name="lower_leg_4_iyy" value="1.914337e-04"/>
+      <xacro:property name="lower_leg_4_iyz" value="8.346770e-06"/>
+      <xacro:property name="lower_leg_4_izz" value="3.656178e-04"/>
       <!-- CECHY POŁOŻENIA STAWÓW LEG 5 -->
       <xacro:property name="joint1_5_xyz" value="-0.121845	0	0.0170504"/>
@@ -320,22 +320,22 @@
       <xacro:property name="link_tip_5_rpy" value="0 0 3.141592654"/>
       <!-- CECHY INERCJI LINKÓW LEG 5 -->
-      <xacro:property name="upper_leg_5_ixx" value="0.000012901"/>
-      <xacro:property name="upper_leg_5_ixy" value="0"/>
-      <xacro:property name="upper_leg_5_ixz" value="0"/>
-      <xacro:property name="upper_leg_5_iyy" value="0.000044860"/>
-      <xacro:property name="upper_leg_5_iyz" value="0"/>
-      <xacro:property name="upper_leg_5_izz" value="0.000047692"/>
-      <xacro:property name="mid_leg_5_ixx" value="0.000064165"/>
-      <xacro:property name="mid_leg_5_ixy" value="0"/>
-      <xacro:property name="mid_leg_5_ixz" value="0"/>
-      <xacro:property name="mid_leg_5_iyy" value="0.000348459"/>
-      <xacro:property name="mid_leg_5_iyz" value="0"/>
-      <xacro:property name="mid_leg_5_izz" value="0.000329761"/>
-      <xacro:property name="lower_leg_5_ixx" value="0.000015420"/>
-      <xacro:property name="lower_leg_5_ixy" value="0"/>
-      <xacro:property name="lower_leg_5_ixz" value="0"/>
-      <xacro:property name="lower_leg_5_iyy" value="0.000337500"/>
-      <xacro:property name="lower_leg_5_iyz" value="0"/>
-      <xacro:property name="lower_leg_5_izz" value="0.000339420"/>
+      <xacro:property name="upper_leg_5_ixx" value="1.365355e-05"/>
+      <xacro:property name="upper_leg_5_ixy" value="-9.739963e-08"/>
+      <xacro:property name="upper_leg_5_ixz" value="1.865460e-07"/>
+      <xacro:property name="upper_leg_5_iyy" value="4.999284e-05"/>
+      <xacro:property name="upper_leg_5_iyz" value="-9.227461e-08"/>
+      <xacro:property name="upper_leg_5_izz" value="5.413814e-05"/>
+      <xacro:property name="mid_leg_5_ixx" value="6.454984e-05"/>
+      <xacro:property name="mid_leg_5_ixy" value="1.702660e-08"/>
+      <xacro:property name="mid_leg_5_ixz" value="-8.257650e-08"/>
+      <xacro:property name="mid_leg_5_iyy" value="3.099780e-04"/>
+      <xacro:property name="mid_leg_5_iyz" value="-2.569593e-08"/>
+      <xacro:property name="mid_leg_5_izz" value="2.854108e-04"/>
+      <xacro:property name="lower_leg_5_ixx" value="1.722692e-05"/>
+      <xacro:property name="lower_leg_5_ixy" value="-2.726535e-08"/>
+      <xacro:property name="lower_leg_5_ixz" value="1.181289e-05"/>
+      <xacro:property name="lower_leg_5_iyy" value="3.656948e-04"/>
+      <xacro:property name="lower_leg_5_iyz" value="-8.782921e-09"/>
+      <xacro:property name="lower_leg_5_izz" value="3.656178e-04"/>
       <!-- CECHY POŁOŻENIA STAWÓW LEG 6 -->
       <xacro:property name="joint1_6_xyz" value="-0.0859957	0.0860903	0.0170505"/>
@@ -358,22 +358,22 @@
       <xacro:property name="link_tip_6_rpy" value="0 0 2.35619449"/>
       <!-- CECHY INERCJI LINKÓW LEG 6 -->
-      <xacro:property name="upper_leg_6_ixx" value="0.000028881"/>
-      <xacro:property name="upper_leg_6_ixy" value="0.000015979"/>
-      <xacro:property name="upper_leg_6_ixz" value="0"/>
-      <xacro:property name="upper_leg_6_iyy" value="0.000028881"/>
-      <xacro:property name="upper_leg_6_iyz" value="0"/>
-      <xacro:property name="upper_leg_6_izz" value="0.000047692"/>
-      <xacro:property name="mid_leg_6_ixx" value="0.000206312"/>
-      <xacro:property name="mid_leg_6_ixy" value="0.000142147"/>
-      <xacro:property name="mid_leg_6_ixz" value="0"/>
-      <xacro:property name="mid_leg_6_iyy" value="0.000206312"/>
-      <xacro:property name="mid_leg_6_iyz" value="0"/>
-      <xacro:property name="mid_leg_6_izz" value="0.000329761"/>
-      <xacro:property name="lower_leg_6_ixx" value="0.000176460"/>
-      <xacro:property name="lower_leg_6_ixy" value="0.000161040"/>
-      <xacro:property name="lower_leg_6_ixz" value="0"/>
-      <xacro:property name="lower_leg_6_iyy" value="0.000176460"/>
-      <xacro:property name="lower_leg_6_iyz" value="0"/>
-      <xacro:property name="lower_leg_6_izz" value="0.000339420"/>
+      <xacro:property name="upper_leg_6_ixx" value="3.172579e-05"/>
+      <xacro:property name="upper_leg_6_ixy" value="1.816965e-05"/>
+      <xacro:property name="upper_leg_6_ixz" value="6.665998e-08"/>
+      <xacro:property name="upper_leg_6_iyy" value="3.192060e-05"/>
+      <xacro:property name="upper_leg_6_iyz" value="-1.971554e-07"/>
+      <xacro:property name="upper_leg_6_izz" value="5.413815e-05"/>
+      <xacro:property name="mid_leg_6_ixx" value="1.872811e-04"/>
+      <xacro:property name="mid_leg_6_ixy" value="1.227142e-04"/>
+      <xacro:property name="mid_leg_6_ixz" value="-7.655812e-08"/>
+      <xacro:property name="mid_leg_6_iyy" value="1.872470e-04"/>
+      <xacro:property name="mid_leg_6_iyz" value="4.021840e-08"/>
+      <xacro:property name="mid_leg_6_izz" value="2.854111e-04"/>
+      <xacro:property name="lower_leg_6_ixx" value="1.914336e-04"/>
+      <xacro:property name="lower_leg_6_ixy" value="1.742339e-04"/>
+      <xacro:property name="lower_leg_6_ixz" value="8.346770e-06"/>
+      <xacro:property name="lower_leg_6_iyy" value="1.914881e-04"/>
+      <xacro:property name="lower_leg_6_iyz" value="-8.359189e-06"/>
+      <xacro:property name="lower_leg_6_izz" value="3.656177e-04"/>
     </xacro:if>
     <xacro:property
