Commit message: Yesterdays deleted commitsCo-authored-by: JuliaHry < JuliaHry@users.noreply.github.com>

File: sim_and_real/ros2_ws_hex/src/hexapod_description/collision/Version2/tip_hitbox.xacro (robot description, xacro)
@@ -16,5 +16,5 @@
         <xacro:property name="sphere_0_radius" value="0.00600"/>
         <!-- <xacro:property name="sphere_0_offset_x" value="0.00000"/> ORYGINALNA WARTOŚĆ -->
-        <xacro:property name="sphere_0_offset_x" value="-0.0025"/> <!--TUTAJ ZMNIEJSZAMY [M] ABY DODAĆ PRZESUNIĘCIE SYMULUJĄCE ODGIĘCIE SPRĘŻYNY -->
+        <xacro:property name="sphere_0_offset_x" value="0.0025"/> <!--TUTAJ ZMNIEJSZAMY [M] ABY DODAĆ PRZESUNIĘCIE SYMULUJĄCE ODGIĘCIE SPRĘŻYNY -->
         <xacro:property name="sphere_0_offset_y" value="0.00000"/> <!--NA RAZIE JEST 0.5CM -->
         <xacro:property name="sphere_0_offset_z" value="0.00000"/>

Commit message: I removed all unnecessary files and organized the packages better.

File: sim_and_real/ros2_ws_hex/src/hexapod_description/collision/Version2/tip_hitbox.xacro (robot description, xacro)
@@ -16,5 +16,5 @@
         <xacro:property name="sphere_0_radius" value="0.00600"/>
         <!-- <xacro:property name="sphere_0_offset_x" value="0.00000"/> ORYGINALNA WARTOŚĆ -->
-        <xacro:property name="sphere_0_offset_x" value="0.0025"/> <!--TUTAJ ZMNIEJSZAMY [M] ABY DODAĆ PRZESUNIĘCIE SYMULUJĄCE ODGIĘCIE SPRĘŻYNY -->
+        <xacro:property name="sphere_0_offset_x" value="0.0"/> <!--TUTAJ ZMNIEJSZAMY [M] ABY DODAĆ PRZESUNIĘCIE SYMULUJĄCE ODGIĘCIE SPRĘŻYNY, było -0.0025 -->
         <xacro:property name="sphere_0_offset_y" value="0.00000"/> <!--NA RAZIE JEST 0.5CM -->
         <xacro:property name="sphere_0_offset_z" value="0.00000"/>

File: sim_and_real/ros2_ws_hex/src/hexapod_description/gazebo/hexapod.gazebo.xacro (robot description, xacro)
@@ -16,10 +16,24 @@
   <xacro:macro name="Link" params="reference">
     <gazebo reference="${reference}">
-      <kp>1000000.0</kp>
-      <kd>100.0</kd>
-      <mu1>0.7</mu1>
-      <mu2>0.7</mu2>
-      <maxVel>1.0</maxVel>
-      <minDepth>0.001</minDepth>
+        <!-- <collision>
+            <surface>
+                <friction>
+                    <ode>
+                        <mu>0.7</mu>
+                        <mu2>0.7</mu2>
+                    </ode>
+                </friction>
+                <contact>
+                    <ode>
+                        <kp>800.0</kp>
+                        <kd>5.0</kd>
+                        <min_depth>0.0</min_depth>
+                        <max_vel>1.0</max_vel>
+                        <soft_cfm>0.02</soft_cfm>
+                        <soft_erp>0.1</soft_erp>
+                    </ode>
+                </contact>
+            </surface>
+        </collision> -->
     </gazebo>
   </xacro:macro>
@@ -27,10 +41,22 @@
    <xacro:macro name="EndEffectorLink" params="reference index">
     <gazebo reference="${reference}">
-      <kp>1000000.0</kp>
-      <kd>100.0</kd>
-      <mu1>0.7</mu1>
-      <mu2>0.7</mu2>
-      <maxVel>1.0</maxVel>
-      <minDepth>0.001</minDepth>
+        <collision>
+            <surface>
+                <friction>
+                    <ode>
+                        <mu>0.7</mu>
+                        <mu2>0.7</mu2>
+                    </ode>
+                </friction>
+                <contact>
+                    <ode>
+                        <kp>820.0</kp>
+                        <kd>100.0</kd>
+                        <min_depth>0.0</min_depth>
+                        <max_vel>1.0</max_vel>
+                    </ode>
+                </contact>
+            </surface>
+        </collision>
     </gazebo>
     <gazebo reference="${prefix}link4_${index}">

File: sim_and_real/ros2_ws_hex/src/hexapod_description/urdf/hexapod_ee.urdf.xacro (robot description, xacro)
@@ -4,7 +4,6 @@
     <xacro:include filename="$(find hexapod_description)/gazebo/hexapod.gazebo.xacro" />
     <xacro:include filename="$(find hexapod_description)/urdf/hexapod_leg_ee.urdf.xacro" />
-    <!-- <xacro:include filename="$(find hexapod_description)/urdf/hexapod_gazebo.urdf.xacro" /> -->
     <xacro:include filename="$(find hexapod_description)/urdf/imu.urdf.xacro"/>
-    <xacro:include filename="$(find hexapod_moveit_config)/config/hexapod.ros2_control.xacro" />
+    <xacro:include filename="$(find hexapod_description)/control/hexapod.ros2_control.xacro" />
     <xacro:hexapod_leg_ee prefix="${prefix}" version="${version}"/>
     <xacro:hexapod_gazebo prefix="${prefix}" />
@@ -19,5 +18,5 @@
     <gazebo>
       <plugin filename="gz_ros2_control-system" name="gz_ros2_control::GazeboSimROS2ControlPlugin">
-        <parameters>$(find hex_gz)/config/gazebo_controller_manager.yaml</parameters>
+        <parameters>$(find hexapod_description)/control/controller_manager.yaml</parameters>
       </plugin>
     </gazebo>
